File: small_led_a/small_led_a.kicad_sch (KiCad schematic)
At the start: 105 parts

Commit message: Update
Parts:
- removed D100, D101, D102, D103, D104, D105, D80, D81, D82, D83, D84, D85, D86, D87, D88, D89, D90, D91, D92, D93, D94, D95, D96, D97, D98, D99: LED, symbol Device:LED
- added D106: LED, LED_SMD:LED_0402_1005Metric, symbol Device:LED
- D1, D10, D11, D12, D13, D14, D15, D16, D17, D18, D19, D2, D20, D21, D22, D23, D24, D25, D26, D27, D28, D29, D3, D30, D31, D32, D33, D34, D35, D36, D37, D38, D39, D4, D40, D41, D42, D43, D44, D45, D46, D47, D48, D49, D5, D50, D51, D52, D53, D54, D55, D56, D57, D58, D59, D6, D60, D61, D62, D63, D64, D65, D66, D67, D68, D69, D7, D70, D71, D72, D73, D74, D75, D76, D77, D78, D79, D8, D9: footprint (none) -> LED_SMD:LED_0402_1005Metric
Connections:
- net k1: now reaches D2.1 (K)
- net k1: now also D1.1 (K), D3.1 (K), D4.1 (K), D5.1 (K), D6.1 (K), D7.1 (K), D106.1 (K)
- net g: now reaches D2.2 (A)
- net g: now also D11.2 (A), D19.2 (A), D27.2 (A), D35.2 (A), D43.2 (A), D51.2 (A), D59.2 (A), D67.2 (A), D75.2 (A)
- net d: now reaches D6.2 (A)
- net d: now also D12.2 (A), D20.2 (A), D28.2 (A), D36.2 (A), D44.2 (A), D52.2 (A), D60.2 (A), D68.2 (A), D76.2 (A)
- net k7: now reaches D48.1 (K)
- net k7: now also D49.1 (K), D50.1 (K), D51.1 (K), D52.1 (K), D53.1 (K), D54.1 (K), D55.1 (K)
- net f: now reaches D48.2 (A)
- net f: now also D16.2 (A), D24.2 (A), D3.2 (A), D32.2 (A), D40.2 (A), D56.2 (A), D64.2 (A), D72.2 (A), D8.2 (A)
- net k8: now reaches D59.1 (K)
- net k8: now also D56.1 (K), D57.1 (K), D58.1 (K), D60.1 (K), D61.1 (K), D62.1 (K), D63.1 (K)
- net k9: now reaches D66.1 (K)
- net k9: now also D64.1 (K), D65.1 (K), D67.1 (K), D68.1 (K), D69.1 (K), D70.1 (K), D71.1 (K)
- net a: now reaches D66.2 (A)
- net a: now also D10.2 (A), D18.2 (A), D26.2 (A), D34.2 (A), D42.2 (A), D50.2 (A), D58.2 (A), D7.2 (A), D74.2 (A)
- net c: now reaches D54.2 (A)
- net c: now also D14.2 (A), D22.2 (A), D30.2 (A), D38.2 (A), D4.2 (A), D46.2 (A), D62.2 (A), D70.2 (A), D78.2 (A)
- net k5: now reaches D39.1 (K)
- net k5: now also D32.1 (K), D33.1 (K), D34.1 (K), D35.1 (K), D36.1 (K), D37.1 (K), D38.1 (K)
- net h: now reaches D39.2 (A)
- net h: now also D15.2 (A), D23.2 (A), D31.2 (A), D47.2 (A), D55.2 (A), D63.2 (A), D71.2 (A), D79.2 (A), D106.2 (A)
- net k10: now reaches D72.1 (K)
- net k10: now also D73.1 (K), D74.1 (K), D75.1 (K), D76.1 (K), D77.1 (K), D78.1 (K), D79.1 (K)
- net k3: now reaches D17.1 (K)
- net k3: now also D16.1 (K), D18.1 (K), D19.1 (K), D20.1 (K), D21.1 (K), D22.1 (K), D23.1 (K)
- net e: now reaches D17.2 (A)
- net e: now also D25.2 (A), D33.2 (A), D41.2 (A), D49.2 (A), D5.2 (A), D57.2 (A), D65.2 (A), D73.2 (A), D9.2 (A)
- net b: now reaches D21.2 (A)
- net b: now also D1.2 (A), D13.2 (A), D29.2 (A), D37.2 (A), D45.2 (A), D53.2 (A), D61.2 (A), D69.2 (A), D77.2 (A)
- net k6: now reaches D42.1 (K)
- net k6: now also D40.1 (K), D41.1 (K), D43.1 (K), D44.1 (K), D45.1 (K), D46.1 (K), D47.1 (K)
- net k4: now reaches D29.1 (K)
- net k4: now also D24.1 (K), D25.1 (K), D26.1 (K), D27.1 (K), D28.1 (K), D30.1 (K), D31.1 (K)
- net k2: now reaches D12.1 (K)
- net k2: now also D10.1 (K), D11.1 (K), D13.1 (K), D14.1 (K), D15.1 (K), D8.1 (K), D9.1 (K)
Other:
- added sheet Untitled Sheet (untitled.kicad_sch)

Commit message: Update
Parts:
- removed D1, D10, D106, D11, D12, D13, D14, D15, D16, D17, D18, D19, D2, D20, D21, D22, D23, D24, D25, D26, D27, D28, D29, D3, D30, D31, D32, D33, D34, D35, D36, D37, D38, D39, D4, D40, D41, D42, D43, D44, D45, D46, D47, D48, D49, D5, D50, D51, D52, D53, D54, D55, D56, D57, D58, D59, D6, D60, D61, D62, D63, D64, D65, D66, D67, D68, D69, D7, D70, D71, D72, D73, D74, D75, D76, D77, D78, D79, D8, D9: LED, LED_SMD:LED_0402_1005Metric, symbol Device:LED
- added J1: Conn_01x23_Pin, Connector_PinHeader_1.27mm:PinHeader_1x23_P1.27mm_Vertical, symbol Connector:Conn_01x23_Pin
- added U1, U10, U11, U12, U13, U14, U15, U2, U3, U4, U5, U6, U7, U8, U9: ~, ajm:seg7_0402, symbol ajm:seg7
Connections:
- net a: now also J1.1 (Pin_1), U1.a, U10.a, U11.a, U12.a, U13.a, U14.a, U15.a, U2.a, U3.a, U4.a, U5.a, U6.a, U7.a, U8.a, U9.a
- net b: now also J1.2 (Pin_2), U1.b, U10.b, U11.b, U12.b, U13.b, U14.b, U15.b, U2.b, U3.b, U4.b, U5.b, U6.b, U7.b, U8.b, U9.b
- net c: now also J1.3 (Pin_3), U1.c, U10.c, U11.c, U12.c, U13.c, U14.c, U15.c, U2.c, U3.c, U4.c, U5.c, U6.c, U7.c, U8.c, U9.c
- net d: now also J1.4 (Pin_4), U1.d, U10.d, U11.d, U12.d, U13.d, U14.d, U15.d, U2.d, U3.d, U4.d, U5.d, U6.d, U7.d, U8.d, U9.d
- net e: now also J1.5 (Pin_5), U1.e, U10.e, U11.e, U12.e, U13.e, U14.e, U15.e, U2.e, U3.e, U4.e, U5.e, U6.e, U7.e, U8.e, U9.e
- net f: now also J1.6 (Pin_6), U1.f, U10.f, U11.f, U12.f, U13.f, U14.f, U15.f, U2.f, U3.f, U4.f, U5.f, U6.f, U7.f, U8.f, U9.f
- net g: now also J1.7 (Pin_7), U1.g, U10.g, U11.g, U12.g, U13.g, U14.g, U15.g, U2.g, U3.g, U4.g, U5.g, U6.g, U7.g, U8.g, U9.g
- net h: now also J1.8 (Pin_8), U1.h, U10.h, U11.h, U12.h, U13.h, U14.h, U15.h, U2.h, U3.h, U4.h, U5.h, U6.h, U7.h, U8.h, U9.h
- net k1: now also J1.9 (Pin_9), U1.k
- net k10: now also J1.18 (Pin_18), U10.k
- net k2: now also J1.10 (Pin_10), U2.k
- net k3: now also J1.11 (Pin_11), U3.k
- net k4: now also J1.12 (Pin_12), U4.k
- net k5: now also J1.13 (Pin_13), U5.k
- net k6: now also J1.14 (Pin_14), U6.k
- net k7: now also J1.15 (Pin_15), U7.k
- net k8: now also J1.16 (Pin_16), U8.k
- net k9: now also J1.17 (Pin_17), U9.k
- new net k11: J1.19 (Pin_19), U11.k
- new net k12: J1.20 (Pin_20), U12.k
- new net k13: J1.21 (Pin_21), U13.k
- new net k14: J1.22 (Pin_22), U14.k
- new net k15: J1.23 (Pin_23), U15.k
Other:
- removed sheet Untitled Sheet
